File: nixie-clock v3/board1.sch (EAGLE design)
At the start: 29 parts, among them IC1 74HC573N, IC2 74HC573N, IC3 74HC573N, IC4 74HC573N, IC5 74HC573N, IC6 74HC573N

Commit message: lots of board progress
Parts:
- removed U$2: MAX1771_NIXIE_MODULE, random:MAX1771_NIXIE_MODULE
- added C1, C2: (no value), resistor-mod:CPOL-EUE3.5-8
- added C3, C4, C6: (no value), resistor:C-EU025-024X044
- added C5: (no value), capacitor-wima:C7.5/5
- added D7: (no value), diode:SCHOTTKY-DIODEDO35-7
- added L1: (no value), inductor-neosid-mod:BS11
- added Q1: IRF620, transistor-fet:IRF620
- added R1: (no value), resistor:R-EU_0309/12
- added R2: 1M5, rcl:R-EU_0204/7
- added R3: 10k, rcl:R-EU_0204/7
- added R4: 5k, resistor:R-TRIMM3296W
- added U$3: MAX1771, maxim:MAX1771
- D1, D2, D3, D4, D5, D6: device diode:DIODE-D-7.5 -> diode-mod:DIODE-D-7.5
- IC1, IC2, IC3, IC4, IC5, IC6: device 74xx-eu:74HC573N -> 74xx-eu-mod:74HC573N
- IC10, IC11, IC7, IC8, IC9: device uln-udn:ULN2803A -> uln-udn-mod:ULN2803ADIL18-ROUND
- IC12: device uln-udn:ULN2803A -> uln-udn-mod:ULN2803ADIL18-ROUND; SPICEPREFIX (none) -> X
- J1: value (none) -> NEB21R; device con-jack:JACK-PLUG0 -> con-lumberg:NEB21R
- SV1, SV2, SV3, SV4, SV5, SV6: device con-lstb:MA08-1 -> con-lstb-mod:MA08-1
Connections:
- removed net N$101: SV7.1, SV7.2, SV7.3, U$2.HV
- new net HV: C1.+, C5.1, D7.C, R2.2, SV7.1, SV7.2, SV7.3
- new net N$105: C4.1, U$3.REF
- new net N$107: Q1.G, U$3.EXT
- new net N$109: D7.A, L1.2, Q1.D
- new net N$110: Q1.S, R1.2, U$3.CS
- new net N$112: R2.1, R4.A, U$3.FB
- new net N$113: R3.2, R4.E, R4.S
- new net SHDN: ARDUINO_NANO1.D13, U$3.SHDN
- net +12V: now also C2.+, C3.1, C6.1, L1.1, U$3.VCC; no longer U$2.VIN
- net GND: now also C1.-, C2.-, C3.2, C4.2, C5.2, C6.2, R1.1, R3.1, U$3.AGND, U$3.GND; no longer U$2.GND, U$2.GND_OUT
Other:
- moved on the sheet: SV7
